File: 7-saw/controller/7-saw-controller w logo and ground plane.brd (EAGLE design)
At the start: 100 x 65 mm, 133 parts, among them IC1 TL074D, IC10 TL072D, IC11 TL074D, IC2 TL074D, IC3 TL072D, IC4 TL074D, IC5 TL074D, IC6 TL074D, IC7 TL074D, IC8 AD633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

Commit message: updated 7-saw
Connections:
- net CENTER_OSC: now also VCA.11; no longer VCA.12
- net SIDE_MIX_SLOPE: now also VCA.12; no longer VCA.11
- net TRIM1+: now also VCA.8; no longer VCA.7
- net TRIM2-: now also VCA.7; no longer VCA.8
Routing:
- net SIDE_MIX_SLOPE: track 18.6 -> 21.3 mm
- net CENTER_OSC: track 18.4 -> 20.9 mm
- net GND: track 692.5 -> 690.4 mm
- net TRIM1+: track 7.47 -> 5.66 mm
- net GNDIO: track 266.5 -> 265.2 mm
- net TRIM2-: track 6.72 -> 5.67 mm
- added copper zone on layer 1, net GND
- added copper zone on layer 16, net GND
Other:
- board text removed: "XONIK DEVICES"
