File: 7-saw/controller/7-saw-controller w logo and ground plane.sch (EAGLE design)
At the start: 133 parts, among them IC1 TL074D, IC10 TL072D, IC11 TL074D, IC2 TL074D, IC3 TL072D, IC4 TL074D, IC5 TL074D, IC6 TL074D, IC7 TL074D, IC8 AD633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

Commit message: updated 7-saw
Connections:
- net CENTER_OSC: now also VCA.11; no longer VCA.12
- net SIDE_MIX_SLOPE: now also VCA.12; no longer VCA.11
- net TRIM1+: now also VCA.8; no longer VCA.7
- net TRIM2-: now also VCA.7; no longer VCA.8
Changed lines of the file:
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@@
 </segment>
 <segment>
-<pinref part="VCA" gate="G$1" pin="11"/>
-<wire x1="261.62" y1="-76.2" x2="284.48" y2="-76.2" width="0.1524" layer="91"/>
-<label x="264.16" y="-76.2" size="1.778" layer="95"/>
+<pinref part="VCA" gate="G$1" pin="12"/>
+<wire x1="261.62" y1="-73.66" x2="284.48" y2="-73.66" width="0.1524" layer="91"/>
+<label x="264.16" y="-73.66" size="1.778" layer="95"/>
 </segment>
 </net>
@@
 </segment>
 <segment>
-<pinref part="VCA" gate="G$1" pin="12"/>
-<wire x1="261.62" y1="-73.66" x2="284.48" y2="-73.66" width="0.1524" layer="91"/>
-<label x="264.16" y="-73.66" size="1.778" layer="95"/>
+<pinref part="VCA" gate="G$1" pin="11"/>
+<wire x1="261.62" y1="-76.2" x2="284.48" y2="-76.2" width="0.1524" layer="91"/>
+<label x="264.16" y="-76.2" size="1.778" layer="95"/>
 </segment>
 </net>
@@
 <net name="TRIM2-" class="0">
 <segment>
-<pinref part="VCA" gate="G$1" pin="8"/>
-<wire x1="261.62" y1="-83.82" x2="294.64" y2="-83.82" width="0.1524" layer="91"/>
-<wire x1="294.64" y1="-83.82" x2="299.72" y2="-88.9" width="0.1524" layer="91"/>
+<pinref part="VCA" gate="G$1" pin="7"/>
+<wire x1="261.62" y1="-86.36" x2="294.64" y2="-86.36" width="0.1524" layer="91"/>
+<wire x1="294.64" y1="-86.36" x2="299.72" y2="-88.9" width="0.1524" layer="91"/>
 <label x="264.16" y="-83.82" size="1.778" layer="95"/>
 <pinref part="R95" gate="G$1" pin="A"/>
@@
 <net name="TRIM1+" class="0">
 <segment>
-<pinref part="VCA" gate="G$1" pin="7"/>
-<wire x1="261.62" y1="-86.36" x2="299.72" y2="-86.36" width="0.1524" layer="91"/>
+<pinref part="VCA" gate="G$1" pin="8"/>
+<wire x1="261.62" y1="-83.82" x2="299.72" y2="-83.82" width="0.1524" layer="91"/>
 <label x="264.16" y="-86.36" size="1.778" layer="95"/>
 <pinref part="R94" gate="G$1" pin="E"/>
-<wire x1="299.72" y1="-81.28" x2="299.72" y2="-86.36" width="0.1524" layer="91"/>
-</segment>
-</net>
+<wire x1="299.72" y1="-81.28" x2="299.72" y2="-83.82" width="0.1524" layer="91"/>
+</segment>
+</net>
